File: _PCB/ESP8266.sch (EAGLE design)
At the start: 46 parts, among them IC1 FT232RL, IC2 LD117AS33TR, Q1 12M, T1 S8050, T2 S8050, X1 MINI-USB-32005-201

Commit message: fix transistor pin E/B swap process
Parts:
- T1, T2: device transistor:-NPN-SOT23-EBC -> transistor:MMBT2222ALT1-NPN-SOT23-BEC
Changed lines of the file:
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@@
 <part name="C9" library="rcl" deviceset="C-US" device="C0805" value="0.1uF"/>
 <part name="C10" library="rcl" deviceset="C-US" device="C0805" value="47uF"/>
-<part name="T1" library="transistor" deviceset="*-NPN-" device="SOT23-EBC" value="S8050"/>
-<part name="T2" library="transistor" deviceset="*-NPN-" device="SOT23-EBC" value="S8050"/>
+<part name="T1" library="transistor" deviceset="*-NPN-" device="SOT23-BEC" technology="MMBT2222ALT1" value="S8050"/>
+<part name="T2" library="transistor" deviceset="*-NPN-" device="SOT23-BEC" technology="MMBT2222ALT1" value="S8050"/>
 <part name="Q1" library="crystal" deviceset="CRYSTAL" device="SM49" value="12M"/>
 <part name="GND" library="supply2" deviceset="GND" device=""/>
@@
 <segment>
 <pinref part="R7" gate="G$1" pin="2"/>
-<wire x1="157.48" y1="71.12" x2="157.48" y2="66.04" width="0.1524" layer="91"/>
-<wire x1="157.48" y1="66.04" x2="162.56" y2="60.96" width="0.1524" layer="91"/>
-<pinref part="T2" gate="G$1" pin="E"/>
-<wire x1="162.56" y1="60.96" x2="172.72" y2="60.96" width="0.1524" layer="91"/>
 <pinref part="IC1" gate="1" pin="!RTS"/>
 <wire x1="127" y1="81.28" x2="157.48" y2="81.28" width="0.1524" layer="91"/>
 <wire x1="157.48" y1="81.28" x2="157.48" y2="71.12" width="0.1524" layer="91"/>
+<pinref part="T2" gate="G$1" pin="E"/>
+<wire x1="172.72" y1="60.96" x2="162.56" y2="60.96" width="0.1524" layer="91"/>
+<wire x1="162.56" y1="60.96" x2="157.48" y2="66.04" width="0.1524" layer="91"/>
+<wire x1="157.48" y1="66.04" x2="157.48" y2="71.12" width="0.1524" layer="91"/>
 <junction x="157.48" y="71.12"/>
 </segment>
@@
 <net name="N$18" class="0">
 <segment>
-<pinref part="T1" gate="G$1" pin="E"/>
-<wire x1="172.72" y1="66.04" x2="162.56" y2="66.04" width="0.1524" layer="91"/>
-<wire x1="162.56" y1="66.04" x2="157.48" y2="60.96" width="0.1524" layer="91"/>
 <pinref part="R8" gate="G$1" pin="2"/>
-<wire x1="157.48" y1="60.96" x2="157.48" y2="55.88" width="0.1524" layer="91"/>
 <pinref part="IC1" gate="1" pin="!DTR"/>
 <wire x1="127" y1="76.2" x2="154.94" y2="76.2" width="0.1524" layer="91"/>
 <wire x1="154.94" y1="76.2" x2="154.94" y2="55.88" width="0.1524" layer="91"/>
 <wire x1="154.94" y1="55.88" x2="157.48" y2="55.88" width="0.1524" layer="91"/>
+<pinref part="T1" gate="G$1" pin="E"/>
+<wire x1="172.72" y1="66.04" x2="162.56" y2="66.04" width="0.1524" layer="91"/>
+<wire x1="162.56" y1="66.04" x2="157.48" y2="60.96" width="0.1524" layer="91"/>
+<wire x1="157.48" y1="60.96" x2="157.48" y2="55.88" width="0.1524" layer="91"/>
 <junction x="157.48" y="55.88"/>
 </segment>
@@
 </sheet>
 </sheets>
+<errors>
+</errors>
 </schematic>
 </drawing>
